File: mp3.kicad_pcb (KiCad board)
At the start: 2 copper layers, 64 x 85.5 mm, 14 parts, among them J1 Micro_SD_Card, J2 AudioPlug3, J3 Conn_01x04, SW1 SW_Push, SW2 SW_Push, SW3 SW_Push, U1 ESP32-WROOM-32, U2 PCM5100A

Commit message: CAD + pcb
Parts:
- added REF**: MountingHole_5mm, MountingHole:MountingHole_5mm, F.Cu at (164.0, 143.0)
- added REF**: MountingHole_5mm, MountingHole:MountingHole_5mm, F.Cu at (112.5, 143.0)
- added REF**: MountingHole_5mm, MountingHole:MountingHole_5mm, F.Cu at (165.0, 88.0)
Routing:
- net GND: track 196.0 -> 202.5 mm
Other:
- board text added: "Front"
- board text added: "back"

Commit message: pcb_update
added the firmware type c port and a boot/flash button
Parts:
- added Boot1: SW_Push, Button_Switch_THT:SW_PUSH_6mm, F.Cu at (147.5, 107.0)
- added C6: 100nf, Capacitor_THT:C_Disc_D5.0mm_W2.5mm_P5.00mm, F.Cu at (142.5, 126.5)
- added C7: 10μf, Capacitor_THT:CP_Radial_D5.0mm_P2.00mm, F.Cu at (130.0, 113.5)
- added J4: USB_C_Receptacle_USB2.0_16P, Connector_USB:USB_C_Receptacle_GCT_USB4105-xx-A_16P_TopMnt_Horizontal, F.Cu at (151.0, 143.5)
- added R3: 5.1kΩ, Resistor_THT:R_Axial_DIN0207_L6.3mm_D2.5mm_P10.16mm_Horizontal, F.Cu at (156.4, 135.5)
- added R4: 5.1kΩ, Resistor_THT:R_Axial_DIN0207_L6.3mm_D2.5mm_P10.16mm_Horizontal, F.Cu at (138.0, 145.6)
- added R5: 10kΩ, Resistor_THT:R_Axial_DIN0207_L6.3mm_D2.5mm_P10.16mm_Horizontal, F.Cu at (146.8, 103.0)
- added U3: CP2102N-Axx-xQFN24, Package_DFN_QFN:QFN-24-1EP_4x4mm_P0.5mm_EP2.6x2.6mm, F.Cu at (142.8, 131.4)
Connections:
- U1 pad 25: unconnected-(U1-IO0-Pad25) -> /boot
- U1 pad 34: unconnected-(U1-RXD0/IO3-Pad34) -> /3
- U1 pad 35: unconnected-(U1-TXD0/IO1-Pad35) -> /1
Routing:
- net GND: track 202.5 -> 289.9 mm
- net +5V: track 0.00 -> 50.8 mm
- net /1: track 0.00 -> 49.9 mm
- net /3: track 0.00 -> 46.9 mm
- net Net-(U3-D-): track 0.00 -> 23.7 mm
- net Net-(U3-D+): track 0.00 -> 21.9 mm
- net +3V3: track 179.3 -> 198.0 mm
- net /CC1: track 0.00 -> 14.6 mm
- net /boot: track 0.00 -> 13.4 mm
- net /CC2: track 0.00 -> 12.7 mm
- net /SCK: track 44.9 -> 46.1 mm
- net /MISO: track 49.2 -> 50.1 mm
Other:
- board text added: "C6"
- board text added: "Flash / boot"
- board text added: "R3"
- board text added: "R4"
