File: mp3.kicad_sch (KiCad schematic)
At the start: 14 parts, among them J1 Micro_SD_Card, J2 AudioPlug3, J3 Conn_01x04, SW1 SW_Push, SW2 SW_Push, SW3 SW_Push, U1 ESP32-WROOM-32, U2 PCM5100A

Commit message: pcb update
Parts:
- C1, C4: footprint (none) -> Capacitor_THT:C_Disc_D5.0mm_W2.5mm_P5.00mm
- C2, C3: footprint (none) -> Capacitor_THT:CP_Radial_D5.0mm_P2.00mm
- J1: footprint (none) -> Connector_Card:microSD_HC_Molex_104031-0811
- J2: footprint (none) -> Connector_Audio:Jack_3.5mm_CUI_SJ1-3533NG_Horizontal
- J3: footprint (none) -> Connector_PinSocket_2.54mm:PinSocket_1x04_P2.54mm_Vertical
- R1: footprint (none) -> Resistor_THT:R_Axial_DIN0207_L6.3mm_D2.5mm_P10.16mm_Horizontal
- R2: footprint (none) -> Potentiometer_THT:Potentiometer_Alps_RK09K_Single_Vertical
- SW1, SW2, SW3: footprint (none) -> Button_Switch_THT:SW_PUSH_6mm
Connections:
- net GPIO25: now also U1.12 (IO27); no longer U1.10 (IO25)
- net GPIO26: now also U1.10 (IO25); no longer U1.11 (IO26)
- net GPIO27: now also U1.11 (IO26); no longer U1.12 (IO27)
Changed lines of the file:
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@@
 		)
 	)
+	(label "GPIO26"
+		(at 218.44 128.27 0)
+		(effects
+			(font
+				(size 1.27 1.27)
+			)
+			(justify left bottom)
+		)
+	)
 	(label "GPIO25"
 		(at 110.49 67.31 180)
@@
 		)
 	)
-	(label "GPIO26"
-		(at 218.44 130.81 0)
-		(effects
-			(font
-				(size 1.27 1.27)
-			)
-			(justify left bottom)
-		)
-	)
 	(label "SCL"
 		(at 205.74 46.99 270)
@@
 		)
 	)
-	(label "GPIO25"
-		(at 218.44 128.27 0)
-		(effects
-			(font
-				(size 1.27 1.27)
-			)
-			(justify left bottom)
-		)
-	)
-	(label "GPIO27"
-		(at 218.44 133.35 0)
+	(label "GPIO33"
+		(at 218.44 138.43 0)
 		(effects
 			(font
@@
 		)
 	)
-	(label "GPIO33"
-		(at 218.44 138.43 0)
+	(label "GPIO34"
+		(at 218.44 140.97 0)
 		(effects
 			(font
@@
 		)
 	)
-	(label "GPIO34"
-		(at 218.44 140.97 0)
+	(label "SCL"
+		(at 218.44 123.19 0)
 		(effects
 			(font
@@
 		)
 	)
-	(label "SCL"
-		(at 218.44 123.19 0)
+	(label "GPIO27"
+		(at 218.44 130.81 0)
 		(effects
 			(font
@@
 		)
 	)
+	(label "GPIO25"
+		(at 218.44 133.35 0)
+		(effects
+			(font
+				(size 1.27 1.27)
+			)
+			(justify left bottom)
+		)
+	)
 	(label "GPIO26"
 		(at 110.49 72.39 180)
@@
 			)
 		)
-		(property "Footprint" ""
+		(property "Footprint" "Connector_PinSocket_2.54mm:PinSocket_1x04_P2.54mm_Vertical"
 			(at 205.74 41.91 0)
 			(hide yes)
@@
 			)
 		)
-		(property "Footprint" ""
+		(property "Footprint" "Connector_Card:microSD_HC_Molex_104031-0811"
 			(at 22.86 170.18 0)
 			(hide yes)
@@
 			)
 		)
-		(property "Footprint" ""
+		(property "Footprint" "Capacitor_THT:C_Disc_D5.0mm_W2.5mm_P5.00mm"
 			(at 107.95 161.5948 0)
 			(hide yes)
@@
 			)
 		)
-		(property "Footprint" ""
+		(property "Footprint" "Capacitor_THT:CP_Radial_D5.0mm_P2.00mm"
 			(at 56.8452 54.61 0)
 			(hide yes)
@@
 			)
 		)
-		(property "Footprint" ""
+		(property "Footprint" "Button_Switch_THT:SW_PUSH_6mm"
 			(at 270.51 31.75 0)
 			(hide yes)
@@
 			)
 		)
-		(property "Footprint" ""
+		(property "Footprint" "Resistor_THT:R_Axial_DIN0207_L6.3mm_D2.5mm_P10.16mm_Horizontal"
 			(at 88.9 180.848 90)
 			(hide yes)
@@
 			)
 		)
-		(property "Footprint" ""
+		(property "Footprint" "Button_Switch_THT:SW_PUSH_6mm"
 			(at 270.51 50.8 0)
 			(hide yes)
@@
 			)
 		)
-		(property "Footprint" ""
+		(property "Footprint" "Capacitor_THT:C_Disc_D5.0mm_W2.5mm_P5.00mm"
 			(at 155.9052 81.28 0)
 			(hide yes)
@@
 			)
 		)
-		(property "Footprint" ""
+		(property "Footprint" "Capacitor_THT:CP_Radial_D5.0mm_P2.00mm"
 			(at 55.5752 77.47 0)
 			(hide yes)
@@
 			)
 		)
-		(property "Footprint" ""
+		(property "Footprint" "Potentiometer_THT:Potentiometer_Alps_RK09K_Single_Vertical"
 			(at 266.7 82.55 0)
 			(hide yes)
@@
 			)
 		)
-		(property "Footprint" ""
+		(property "Footprint" "Button_Switch_THT:SW_PUSH_6mm"
 			(at 270.51 64.77 0)
 			(hide yes)
@@
 			)
 		)
-		(property "Footprint" ""
+		(property "Footprint" "Connector_Audio:Jack_3.5mm_CUI_SJ1-3533NG_Horizontal"
 			(at 31.75 63.5 0)
 			(hide yes)

Commit message: CAD + pcb
Connections:
- net GPIO16: now also U1.7 (IO35); no longer U1.27 (IO16)
Changed lines of the file:
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@@
-	)
-	(no_connect
-		(at 218.44 143.51)
 	)
 	(no_connect
@@
 	(no_connect
 		(at 218.44 102.87)
+	)
+	(no_connect
+		(at 218.44 110.49)
 	)
 	(no_connect
@@
 		)
 	)
+	(label "GPIO16"
+		(at 218.44 143.51 0)
+		(effects
+			(font
+				(size 1.27 1.27)
+			)
+			(justify left bottom)
+		)
+	)
 	(label "MISO"
 		(at 74.93 154.94 0)
@@
 		(effects
 			(font
-				(size 1.27 1.27)
-			)
-			(justify left bottom)
-		)
-	)
-	(label "GPIO16"
-		(at 218.44 110.49 0)
-		(effects
-			(font

Commit message: гзвфеу
Parts:
- added Boot1: SW_Push, Button_Switch_THT:SW_PUSH_6mm, symbol Switch:SW_Push
- added J4: USB_C_Receptacle_USB2.0_16P, symbol Connector:USB_C_Receptacle_USB2.0_16P
- added R3, R4: 5.1kΩ, symbol Device:R
- added R5: 10kΩ, Resistor_THT:R_Axial_DIN0207_L6.3mm_D2.5mm_P10.16mm_Horizontal, symbol Device:R
- added U3: CP2102N-Axx-xQFN24, Package_DFN_QFN:QFN-24-1EP_4x4mm_P0.5mm_EP2.6x2.6mm, symbol Interface_USB:CP2102N-Axx-xQFN24
Connections:
- net +3V3: now also R5.2, U3.5 (VIO), U3.6 (VDD)
- net GND: now also Boot1.2, J4.A1 (GND), J4.A12 (GND), J4.B1 (GND), J4.B12 (GND), J4.SH (SHIELD), R3.2, R4.2, U3.2 (GND), U3.25 (GND)
- net boot: now reaches U1.25 (IO0)
- net boot: now also Boot1.1, R5.1
- net 3: now reaches U1.34 (RXD0/IO3)
- net 3: now also U3.20 (RXD)
- net 1: now reaches U1.35 (TXD0/IO1)
- net 1: now also U3.21 (TXD)
- new net: J4.A6 (D+), J4.B6 (D+), U3.3 (D+)
- new net: J4.A7 (D-), J4.B7 (D-), U3.4 (D-)
- new net +5V: J4.A4 (VBUS), J4.A9 (VBUS), J4.B4 (VBUS), J4.B9 (VBUS), U3.7 (VREGIN), U3.8 (VBUS)
- new net CC1: J4.A5 (CC1), R3.1
- new net CC2: J4.B5 (CC2), R4.1
- no-connect marks 32 -> 43
Other:
- moved on the sheet: J3, U1

Commit message: pcb_update
added the firmware type c port and a boot/flash button
Parts:
- added C5, C6: 100nf, Capacitor_THT:C_Disc_D5.0mm_W2.5mm_P5.00mm, symbol Device:C
- added C7: 10μf, Capacitor_THT:CP_Radial_D5.0mm_P2.00mm, symbol Device:C_Polarized
- J4: footprint (none) -> Connector_USB:USB_C_Receptacle_GCT_USB4105-xx-A_16P_TopMnt_Horizontal
- R3, R4: footprint (none) -> Resistor_THT:R_Axial_DIN0207_L6.3mm_D2.5mm_P10.16mm_Horizontal
Connections:
- net +3V3: now also C5.1, C6.1, C7.1
- net GND: now also C5.2, C6.2, C7.2
Other:
- moved on the sheet: R4
