File: PCB/mp3.kicad_pcb (KiCad board)
At the start: 2 copper layers, 64 x 85.5 mm, 25 parts, among them J1 Micro_SD_Card, J2 AudioPlug3, J3 Conn_01x04, J4 USB_C_Receptacle_USB2.0_16P, SW1 SW_Push, SW2 SW_Push, SW3 SW_Push, U1 ESP32-WROOM-32, U2 PCM5100A, U3 CP2102N-Axx-xQFN24

Commit message: added battery
Parts:
- added C10: 100μf, Capacitor_SMD:CP_Elec_6.3x5.4, F.Cu at (124.0, 109.5)
- added C5: 100nf, Capacitor_THT:C_Disc_D5.0mm_W2.5mm_P5.00mm, F.Cu at (163.0, 115.0)
- added C8: 10μf, Capacitor_SMD:C_0805_2012Metric, F.Cu at (166.5, 105.0)
- added C9: 10μf, Capacitor_SMD:C_0805_2012Metric, F.Cu at (163.0, 103.0)
- added J5: battery, Connector_Molex:Molex_KK-254_AE-6410-02A_1x02_P2.54mm_Vertical, F.Cu at (165.5, 109.0)
- added U4: AP2112K-3.3, Package_TO_SOT_SMD:SOT-23-5, F.Cu at (166.4, 99.0)
Routing:
- net GND: track 289.9 -> 339.9 mm
- net /VBAT: track 0.00 -> 13.2 mm
- net /MOSI: track 51.5 -> 61.8 mm
- net +3V3: track 198.0 -> 203.0 mm
