File: PCB/mp3.kicad_sch (KiCad schematic)
At the start: 23 parts, among them J1 Micro_SD_Card, J2 AudioPlug3, J3 Conn_01x04, J4 USB_C_Receptacle_USB2.0_16P, SW1 SW_Push, SW2 SW_Push, SW3 SW_Push, U1 ESP32-WROOM-32, U2 PCM5100A, U3 CP2102N-Axx-xQFN24

Commit message: added battery
Parts:
- added C10: 100μf, Capacitor_SMD:CP_Elec_6.3x5.4, symbol Device:C
- added C8, C9: 10μf, Capacitor_SMD:C_0805_2012Metric, symbol Device:C
- added J5: battery, Connector_Molex:Molex_KK-254_AE-6410-02A_1x02_P2.54mm_Vertical, symbol Connector_Generic:Conn_01x02
- added U4: AP2112K-3.3, Package_TO_SOT_SMD:SOT-23-5, symbol Regulator_Linear:AP2112K-3.3
Connections:
- net +3V3: now also C10.1, C9.1, U4.5 (VOUT)
- net GND: now also C10.2, C8.2, C9.2, J5.2 (Pin_2), U4.2 (GND)
- new net VBAT: C8.1, J5.1 (Pin_1), U4.1 (VIN), U4.3 (EN)
- no-connect marks 43 -> 44
Other:
- moved on the sheet: Boot1, C5, J4, R3, R4, R5, U3
